File: hardware/asm_led_controller.kicad_pcb (KiCad board)
At the start: 2 copper layers, 199.5 x 92.1 mm, 67 parts, among them J1 Flash Interface, SW1 On/Off Switch ASM, SW2 Frequency Switch, SW3 Run/Flash Switch 1, SW4 Run/Flash Switch 2, SW5 On/Off Switch LED, U1 AS6C1008-55PCN Program Memory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, U2 AS6C1008-55PCN Program Memory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, U3 AS6C1008-55PCN Program Memory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, U4 4060 Frequency Counter, U5 4060 Program Counter, U6 LM7805

Commit message: Readded silkscreen labels
Parts:
- FLASH INTERFACE: renamed from J1
- ON/OFF LED: renamed from SW5
- renumbered SW2 to FREQUENCY, SW1 to ON/OFF, SW4 to RUN/FLASH
Changed lines of the file:
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@@
 		(layer "F.Cu")
 		(at 51.44 132.43 90)
-		(property "Reference" "SW2"
+		(property "Reference" "FREQUENCY"
 			(at 8.4 0 180)
 			(layer "F.SilkS")
@@
 		(at 62.19 128.68)
 		(descr "JS202011CQN DPDT Sub-Miniature Slide Switchwww.ck-components.com")
-		(property "Reference" "SW4"
+		(property "Reference" "RUN/FLASH"
 			(at 0.31 -3.68 0)
 			(layer "F.SilkS")
@@
 		(descr "CuK miniature slide switch, OS series, SPDT, https://www.ckswitches.com/media/1428/os.pdf")
 		(tags "switch SPDT")
-		(property "Reference" "SW1"
+		(property "Reference" "ON/OFF"
 			(at 2.31 -3.28 0)
 			(layer "F.SilkS")
@@
 		(descr "Through hole straight pin header, 2x13, 2.54mm pitch, double rows")
 		(tags "Through hole pin header THT 2x13 2.54mm double row")
-		(property "Reference" "J1"
+		(property "Reference" "FLASH INTERFACE"
 			(at -5.2 -2.78 270)
 			(layer "F.SilkS")
@@
 		(at 62.19 116.13)
 		(descr "JS202011CQN DPDT Sub-Miniature Slide Switchwww.ck-components.com")
-		(property "Reference" "SW5"
+		(property "Reference" "ON/OFF LED"
 			(at 0.31 -3.38 0)
 			(layer "F.SilkS")
@@
 	)
 	(segment
+		(start 43 110)
+		(end 42 109)
+		(width 0.2)
+		(layer "F.Cu")
+		(net "Net-(U4-Q7)")
+	)
+	(segment
+		(start 36.63 108.13)
+		(end 36.63 106.59)
+		(width 0.2)
+		(layer "F.Cu")
+		(net "Net-(U4-Q7)")
+	)
+	(segment
+		(start 51.44 130.43)
+		(end 50.51 129.5)
+		(width 0.2)
+		(layer "F.Cu")
+		(net "Net-(U4-Q7)")
+	)
+	(segment
+		(start 42 109)
+		(end 37.5 109)
+		(width 0.2)
+		(layer "F.Cu")
+		(net "Net-(U4-Q7)")
+	)
+	(segment
+		(start 46.96 129.5)
+		(end 43 125.54)
+		(width 0.2)
+		(layer "F.Cu")
+		(net "Net-(U4-Q7)")
+	)
+	(segment
+		(start 43 125.54)
+		(end 43 110)
+		(width 0.2)
+		(layer "F.Cu")
+		(net "Net-(U4-Q7)")
+	)
+	(segment
+		(start 50.51 129.5)
+		(end 46.96 129.5)
+		(width 0.2)
+		(layer "F.Cu")
+		(net "Net-(U4-Q7)")
+	)
+	(segment
+		(start 37.5 109)
+		(end 36.63 108.13)
+		(width 0.2)
+		(layer "F.Cu")
+		(net "Net-(U4-Q7)")
+	)
+	(segment
 		(start 47.53125 128.43)
 		(end 51.44 128.43)
@@
 	)
 	(segment
+		(start 41.71 114.53)
+		(end 42.04 114.53)
+		(width 0.2)
+		(layer "F.Cu")
+		(net "unconnected-(U4-Q9-Pad13)")
+	)
+	(segment
+		(start 46.84 114.58)
+		(end 46.79 114.53)
+		(width 0.2)
+		(layer "F.Cu")
+		(net "unconnected-(U4-Q10-Pad15)")
+	)
+	(segment
 		(start 214.5 95.5)
 		(end 159.32 95.5)
@@
 		(net "Net-(D8-A)")
 	)
-	(segment
-		(start 43 110)
-		(end 42 109)
-		(width 0.2)
-		(layer "F.Cu")
-		(net "Net-(U4-Q7)")
-	)
-	(segment
-		(start 36.63 108.13)
-		(end 36.63 106.59)
-		(width 0.2)
-		(layer "F.Cu")
-		(net "Net-(U4-Q7)")
-	)
-	(segment
-		(start 51.44 130.43)
-		(end 50.51 129.5)
-		(width 0.2)
-		(layer "F.Cu")
-		(net "Net-(U4-Q7)")
-	)
-	(segment
-		(start 42 109)
-		(end 37.5 109)
-		(width 0.2)
-		(layer "F.Cu")
-		(net "Net-(U4-Q7)")
-	)
-	(segment
-		(start 46.96 129.5)
-		(end 43 125.54)
-		(width 0.2)
-		(layer "F.Cu")
-		(net "Net-(U4-Q7)")
-	)
-	(segment
-		(start 43 125.54)
-		(end 43 110)
-		(width 0.2)
-		(layer "F.Cu")
-		(net "Net-(U4-Q7)")
-	)
-	(segment
-		(start 50.51 129.5)
-		(end 46.96 129.5)
-		(width 0.2)
-		(layer "F.Cu")
-		(net "Net-(U4-Q7)")
-	)
-	(segment
-		(start 37.5 109)
-		(end 36.63 108.13)
-		(width 0.2)
-		(layer "F.Cu")
-		(net "Net-(U4-Q7)")
-	)
-	(segment
-		(start 46.84 114.58)
-		(end 46.79 114.53)
-		(width 0.2)
-		(layer "F.Cu")
-		(net "unconnected-(U4-Q10-Pad15)")
-	)
-	(segment
-		(start 41.71 114.53)
-		(end 42.04 114.53)
-		(width 0.2)
-		(layer "F.Cu")
-		(net "unconnected-(U4-Q9-Pad13)")
-	)
 	(zone

Commit message: Updated frequency switch silkscreen
Other:
- board text added: "FAST"
- board text added: "PAUSE"
- board text added: "SLOW"
- board text removed: "1"
- board text removed: "2"
- board text removed: "3"
Changed lines of the file:
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@@
 		)
 	)
-	(gr_text "1"
-		(at 47.5 129.75 0)
+	(gr_text "PAUSE"
+		(at 44 136.25 0)
 		(layer "F.SilkS")
 		(effects
@@
 		)
 	)
-	(gr_text "2"
-		(at 47.5 133 0)
+	(gr_text "SLOW"
+		(at 44.75 129.75 0)
 		(layer "F.SilkS")
 		(effects
@@
 		)
 	)
-	(gr_text "3"
-		(at 47.5 136.25 0)
+	(gr_text "FAST"
+		(at 45.25 133 0)
 		(layer "F.SilkS")
 		(effects
